Commit message: fix lidar visiual

File: src/robot_control/model/tracked_vehicle.urdf.xacro (robot description, xacro)
@@ -529,91 +529,92 @@
         <!-- <hardwareInterface>hardware_interface/EffortJointInterface</hardwareInterface> -->
     </joint>
-<joint name="velodyne_base_mount_joint" type="fixed">
-    <origin rpy="0 0 0" xyz="0 0 0.2"/>
-    <parent link="base_link"/>
-    <child link="velodyne_base_link"/>
-  </joint>
-  <link name="velodyne_base_link">
-    <inertial>
-      <mass value="0.83"/>
-      <origin xyz="0 0 0.03585"/>
-      <inertia ixx="0.000908059425" ixy="0" ixz="0" iyy="0.000908059425" iyz="0" izz="0.0011049624"/>
-    </inertial>
-    <visual>
-      <geometry>
-        <mesh filename="package://velodyne_description/meshes/VLP16_base_1.dae"/>
-      </geometry>
-    </visual>
-    <visual>
-      <geometry>
-        <mesh filename="package://velodyne_description/meshes/VLP16_base_2.dae"/>
-      </geometry>
-    </visual>
-    <collision>
-      <origin rpy="0 0 0" xyz="0 0 0.03585"/>
-      <geometry>
-        <cylinder length="0.0717" radius="0.0516"/>
-      </geometry>
-    </collision>
-  </link>
-  <joint name="velodyne_base_scan_joint" type="fixed">
-    <origin rpy="0 0 0" xyz="0 0 0.0377"/>
-    <parent link="velodyne_base_link"/>
-    <child link="velodyne"/>
-  </joint>
-  <link name="velodyne">
-    <inertial>
-      <mass value="0.01"/>
-      <origin xyz="0 0 0"/>
-      <inertia ixx="1e-7" ixy="0" ixz="0" iyy="1e-7" iyz="0" izz="1e-7"/>
-    </inertial>
-    <visual>
-      <origin xyz="0 0 -0.0377"/>
-      <geometry>
-        <mesh filename="package://velodyne_description/meshes/VLP16_scan.dae"/>
-      </geometry>
-    </visual>
-  </link>
-  <!-- Gazebo requires the velodyne_gazebo_plugins package -->
-  <gazebo reference="velodyne">
-    <sensor name="velodyne-VLP16" type="ray">
-      <pose>0 0 0 0 0 0</pose>
-      <visualize>false</visualize>
-      <update_rate>10</update_rate>
-      <ray>
-        <scan>
-          <horizontal>
-            <samples>440</samples>
-            <resolution>1</resolution>
-            <min_angle>-3.141592653589793</min_angle>
-            <max_angle>3.141592653589793</max_angle>
-          </horizontal>
-          <vertical>
-            <samples>16</samples>
-            <resolution>1</resolution>
-            <min_angle>-0.2617993877991494</min_angle>
-            <max_angle> 0.2617993877991494</max_angle>
-          </vertical>
-        </scan>
-        <range>
-          <min>0.3</min>
-          <max>131.0</max>
-          <resolution>0.001</resolution>
-        </range>
-        <noise>
-          <type>gaussian</type>
-          <mean>0.0</mean>
-          <stddev>0.0</stddev>
-        </noise>
-      </ray>
-      <plugin filename="libgazebo_ros_velodyne_laser.so" name="gazebo_ros_laser_controller">
-        <topicName>/velodyne_points</topicName>
-        <frameName>velodyne</frameName>
-        <min_range>0.9</min_range>
-        <max_range>130.0</max_range>
-        <gaussianNoise>0.008</gaussianNoise>
-      </plugin>
-    </sensor>
-  </gazebo>
+    <joint name="velodyne_base_mount_joint" type="fixed">
+        <origin rpy="0 0 0" xyz="0 0 0.2" />
+        <parent link="base_link" />
+        <child link="velodyne_base_link" />
+    </joint>
+    <link name="velodyne_base_link">
+        <inertial>
+            <mass value="0.83" />
+            <origin xyz="0 0 0.03585" />
+            <inertia ixx="0.000908059425" ixy="0" ixz="0" iyy="0.000908059425" iyz="0"
+                izz="0.0011049624" />
+        </inertial>
+        <visual>
+            <geometry>
+                <mesh filename="package://velodyne_description/meshes/VLP16_base_1.dae" />
+            </geometry>
+        </visual>
+        <visual>
+            <geometry>
+                <mesh filename="package://velodyne_description/meshes/VLP16_base_2.dae" />
+            </geometry>
+        </visual>
+        <collision>
+            <origin rpy="0 0 0" xyz="0 0 0.03585" />
+            <geometry>
+                <cylinder length="0.0717" radius="0.0516" />
+            </geometry>
+        </collision>
+    </link>
+    <joint name="velodyne_base_scan_joint" type="fixed">
+        <origin rpy="0 0 0" xyz="0 0 0.0377" />
+        <parent link="velodyne_base_link" />
+        <child link="velodyne" />
+    </joint>
+    <link name="velodyne">
+        <inertial>
+            <mass value="0.01" />
+            <origin xyz="0 0 0" />
+            <inertia ixx="1e-7" ixy="0" ixz="0" iyy="1e-7" iyz="0" izz="1e-7" />
+        </inertial>
+        <visual>
+            <origin xyz="0 0 -0.0377" />
+            <geometry>
+                <mesh filename="package://velodyne_description/meshes/VLP16_scan.dae" />
+            </geometry>
+        </visual>
+    </link>
+    <!-- Gazebo requires the velodyne_gazebo_plugins package -->
+    <gazebo reference="velodyne">
+        <sensor name="velodyne-VLP16" type="ray">
+            <pose>0 0 0 0 0 0</pose>
+            <visualize>false</visualize>
+            <update_rate>10</update_rate>
+            <ray>
+                <scan>
+                    <horizontal>
+                        <samples>440</samples>
+                        <resolution>1</resolution>
+                        <min_angle>-3.141592653589793</min_angle>
+                        <max_angle>3.141592653589793</max_angle>
+                    </horizontal>
+                    <vertical>
+                        <samples>16</samples>
+                        <resolution>1</resolution>
+                        <min_angle>-0.2617993877991494</min_angle>
+                        <max_angle> 0.2617993877991494</max_angle>
+                    </vertical>
+                </scan>
+                <range>
+                    <min>0.3</min>
+                    <max>131.0</max>
+                    <resolution>0.001</resolution>
+                </range>
+                <noise>
+                    <type>gaussian</type>
+                    <mean>0.0</mean>
+                    <stddev>0.0</stddev>
+                </noise>
+            </ray>
+            <plugin filename="libgazebo_ros_velodyne_laser.so" name="gazebo_ros_laser_controller">
+                <topicName>/velodyne_points</topicName>
+                <frameName>velodyne</frameName>
+                <min_range>0.9</min_range>
+                <max_range>130.0</max_range>
+                <gaussianNoise>0.008</gaussianNoise>
+            </plugin>
+        </sensor>
+    </gazebo>
     <!-- <xacro:include
     filename="/home/tzh/track-flipper/src/velodyne_simulator/velodyne_description/urdf/VLP-16.urdf.xacro"

Commit message: add imu and flipper control

File: src/robot_control/model/tracked_vehicle.urdf.xacro (robot description, xacro)
@@ -227,5 +227,5 @@
         <child link="front_left_flipper" />
         <!-- 关节相对于父链接的位姿 -->
-        <origin xyz="0.25 0.073545 0.0195" rpy="0 -0.5 0" />
+        <origin xyz="0.25 0.073545 0.0195" rpy="0 -1.57 0" />
         <!-- 旋转轴 -->
         <axis xyz="0 1 0" />
@@ -324,5 +324,5 @@
         <child link="rear_left_flipper" />
         <!-- 关节在父链接坐标系中的位姿 -->
-        <origin xyz="-0.25 0.073545 0.0195" rpy="3.14159 -0.5 3.14159" />
+        <origin xyz="-0.25 0.073545 0.0195" rpy="3.14159 -1.57 0" />
         <!-- 旋转轴 -->
         <axis xyz="0 1 0" />
@@ -422,5 +422,5 @@
         <child link="front_right_flipper" />
         <!-- 关节相对于父链接的位姿 -->
-        <origin xyz="0.25 -0.073545 0.0195" rpy="3.14159 0.5 3.14159" />
+        <origin xyz="0.25 -0.073545 0.0195" rpy="3.14159 1.57 3.14159" />
         <!-- 旋转轴 -->
         <axis xyz="0 1 0" />
@@ -519,5 +519,5 @@
         <child link="rear_right_flipper" />
         <!-- 关节在父链接坐标系中的位姿（根据实际需求修改） -->
-        <origin xyz="-0.25 -0.073545 0.0195" rpy="0 0.5 0" />
+        <origin xyz="-0.25 -0.073545 0.0195" rpy="0 1.57 3.14159" />
         <!-- 旋转轴 -->
         <axis xyz="0 1 0" />
